Commit message: the velocity thing isn't working, the joints are collapsing to the origin when the controllers are launched.

File: src/testbot25_description/urdf/testbot25.xacro (robot description, xacro)
@@ -34,5 +34,5 @@
     <origin xyz="0.00023306481069784724 -0.02318972454000136 -8.598759102573794e-05" rpy="0 0 0"/>
     <mass value="2.3755548141648055"/>
-    <inertia ixx="0.003976" iyy="0.007233" izz="0.003977" ixy="-1.1e-05" iyz="4e-06" ixz="0.0"/>
+    <inertia ixx="0.003976" iyy="0.007233" izz="0.003977" ixy="0.0" iyz="0.0" ixz="0.0"/>
   </inertial>
   <visual>
@@ -54,5 +54,5 @@
     <origin xyz="0.023189720713294504 -4.460789661273057e-05 0.0002442722113514678" rpy="0 0 0"/>
     <mass value="2.3755548141648055"/>
-    <inertia ixx="0.007233" iyy="0.003977" izz="0.003976" ixy="-3e-06" iyz="1e-06" ixz="1.1e-05"/>
+    <inertia ixx="0.007233" iyy="0.003977" izz="0.003976" ixy="0.0" iyz="0.0" ixz="0.0"/>
   </inertial>
   <visual>
@@ -74,5 +74,5 @@
     <origin xyz="-0.00013084904273691356 0.023189727913186076 0.00021110193424155044" rpy="0 0 0"/>
     <mass value="2.3755548141648055"/>
-    <inertia ixx="0.003977" iyy="0.007233" izz="0.003976" ixy="-6e-06" iyz="1e-05" ixz="1e-06"/>
+    <inertia ixx="0.003977" iyy="0.007233" izz="0.003976" ixy="0.0" iyz="0.0" ixz="0.0"/>
   </inertial>
   <visual>
@@ -94,5 +94,5 @@
     <origin xyz="-0.023189726347854874 -1.3442187194345756e-05 -0.00024875241505260826" rpy="0 0 0"/>
     <mass value="2.3755548141648055"/>
-    <inertia ixx="0.007233" iyy="0.003977" izz="0.003976" ixy="1e-06" iyz="-0.0" ixz="1.2e-05"/>
+    <inertia ixx="0.007233" iyy="0.003977" izz="0.003976" ixy="0.0" iyz="-0.0" ixz="0.0"/>
   </inertial>
   <visual>
